File: kicad/main.kicad_pcb (KiCad board)
At the start: 4 copper layers, 44.7 x 52.9 mm, 17 parts, among them J1 Conn_battery, J2 AudioJack3, J3 USB_PWR, SW1 SW_Push, U1 TPS73101DBV, U2 ESP32_DevKit_V1

Commit message: feat: update schematic with protection RC
Parts:
- added C1: 100n, Capacitor_SMD:C_1206_3216Metric, B.Cu at (109.3, 74.7)
- added C2: 100n, Capacitor_SMD:C_1206_3216Metric, B.Cu at (109.5, 80.6)
- added R10: 1k, Resistor_SMD:R_0805_2012Metric, B.Cu at (106.2, 76.3)
- added R11: 1k, Resistor_SMD:R_0805_2012Metric, B.Cu at (106.2, 79.1)
Connections:
- J2 pad R: DAH -> Net-(C2-Pad1)
- J2 pad T: DIT -> Net-(C1-Pad1)
Routing:
- net DIT: track 41.8 -> 3.85 mm
- net Net-(C1-Pad1): track 0.00 -> 36.3 mm
- net DAH: track 38.6 -> 3.84 mm
- net Net-(C2-Pad1): track 0.00 -> 33.3 mm
Other:
- board size 44.7 x 52.9 mm -> 59.8 x 52.9 mm
